File: wenzels-mosfet-class-a-headphones-stereo-amp/wenzels-mosfet-class-a-headphones-stereo-amp.kicad_sch (KiCad schematic)
At the start: 62 parts, among them J1 24V, J3 Input, J4 Headphones out, Q1 K170, Q2 IRFZ44N, Q3 K170, Q4 IRFZ44N, SW1 POWER ON

Commit message: wenzels-mosfet-class-a-headphones-stereo-amp: 2025-11 r2 release
Parts:
- added OUTPUT: B10k, symbol Device:R_Potentiometer_Dual
- R24, R3: value 1k -> 330
- R29, R32: value 47k -> 10k
Connections:
- net GND: now also OUTPUT.1, OUTPUT.4; no longer INPUT.3, J3.R
- net at C15.2, R33.1: no longer R32.1
- net at C13.2: now also OUTPUT.2; no longer C12.2
- net at C22.1, J4.R, R33.2: now also R32.1
- net at C7.2, R12.1: no longer R29.1
- net at C21.1, J4.T, R12.2: now also R29.1
- net at C4.2: now also OUTPUT.5; no longer C6.2
- new net: C12.2, OUTPUT.3
- new net: C6.2, OUTPUT.6
- new net: INPUT.3, J3.R
Other:
- note added: "Better to use A10k (logarithmic) for INPUT and OUTPUT pots but stereo logarithmic ones are harder to find."
- note removed: "Better to use A10k (logarithmic) but stereo logarithmic ones are harder to find."
- moved on the sheet: C13, C14, C15, C4, C7, C9, R12, R24, R29, R3, R33
