File: wenzels-transparent-balancing-opamp-boost/wenzels-transparent-balancing-opamp-boost.kicad_sch (KiCad schematic)
At the start: 82 parts, among them J1 Input-A, J2 Output-A, J3 DC jack 18V, J4 DC jack 18V, J5 Input-B, J6 Output-B, SW1 SOLID/LIFTED CHASSIS GND, SW2 Out-A GND LIFT, SW3 Out-B GND LIFT, SW4 Out-B GND LIFT, SW5 Out-B GND LIFT, U1 NE5532, U2 NE5532, U3 NE5532

Commit message: wenzels-transparent-balancing-opamp-boost: Fix V- power supply filter
Parts:
- removed SW3: Out-B GND LIFT, Button_Switch_SMD:Nidec_Copal_CAS-120A, symbol Switch:SW_Nidec_CAS-120A1
- added SW6: Out-B GND LIFT, Button_Switch_SMD:Nidec_Copal_CAS-120A, symbol Switch:SW_Nidec_CAS-120A1
- SW4: value Out-B GND LIFT -> In-A GND LIFT
- SW5: value Out-B GND LIFT -> In-B GND LIFT
Connections:
- net -18V: no longer C1.2, C10.1, C11.2, C12.2, C13.2, C14.2, C15.2, C16.2, C17.2, C18.2, C19.2, C2.2, C20.2, C21.2, C23.2, C25.2, C26.2, C27.2, C28.1, C29.2, C3.1, C30.1, C31.2, C32.1, C33.2, C4.1, C5.1, C6.2, C7.1, C8.2, C9.2, D1.2 (A), D2.1 (K), D3.1 (K), D4.1 (K), D5.2 (A), D6.2 (A), J3.1, J4.1, R13.2, SW1.2 (B), SW1.3 (A), U1.3 (+), U1.5 (+), U2.3 (+), U2.5 (+), U3.3 (+), U3.5 (+)
- net Chassis: now also SW6.2 (B), SW6.3 (A); no longer J1.S, J5.S, SW4.1 (C), SW5.1 (C)
- net at J6.S: now also SW6.1 (C)
- net at L2.2, R4.2: now also C18.2, C20.2; no longer C18.1, C20.1
- net + renamed GND
- net GND: now also C1.2, C10.1, C11.2, C12.2, C13.2, C14.2, C15.2, C16.2, C17.2, C18.1, C19.2, C2.2, C20.1, C21.2, C23.2, C25.2, C26.2, C27.2, C28.1, C29.2, C3.1, C30.1, C31.2, C32.1, C33.2, C4.1, C5.1, C6.2, C7.1, C8.2, C9.2, D1.2 (A), D2.1 (K), D3.1 (K), D4.1 (K), D5.2 (A), D6.2 (A), J3.1, J4.1, R13.2, SW1.2 (B), SW1.3 (A), U1.3 (+), U1.5 (+), U2.3 (+), U2.5 (+), U3.3 (+), U3.5 (+)
- new net: J1.S, SW4.1 (C)
- new net: J5.S, SW5.1 (C)
Other:
- moved on the sheet: C33, D3, D6, L2, R12, R13, R4, SW1
