File: wenzels-fuzz-boost/wenzels-fuzz-boost.kicad_sch (KiCad schematic)
At the start: 77 parts, among them J1 Input jack, J2 Output jack, J3 18V, Q1 NPN, Q1B B1M, Q2 NPN, Q2B B1M, Q3 J113, Q4 J113, Q5 J113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

Commit message: wenzels-fuzz-boost: r3-wip-2
Parts:
- removed R13: 10k, symbol Device:R
- added C28, C29: 47u, electrolytic, symbol Device:C_Polarized
- added SW2: MORE, symbol Switch:SW_Push_DPDT
Connections:
- net GND: now also SW2.2 (B), SW2.5 (B)
- net at Q2.3 (E), R6.1: now also C29.1
- net at Q1.3 (E), R5.1: now also C28.1
- new net: C28.2, SW2.3 (C)
- new net: C29.2, SW2.6 (C)
- no-connect marks 0 -> 2
Other:
- note added: "Parts (resistors are not listed here): - 6x potentiometers total (2x B1M, A1M, 2x A100k, A10k) - 2x switches (1x DPDT and 1x SPDT) - A bunch of 47u >=25V electrolytic capacitors - A bunch of 100n film capacitors - Ceramic caps: 10p, 100p, 2x of 47p - 2x 4u7 >=25V eletrolytic cap - 1x 3n3 film cap - 2x 1n4007 diodes - 1x 1n5819 diodes"
