File: guitar-preamps/wenzels-fruity-tube-guitar-preamp/wenzels-fruity-tube-guitar-preamp.kicad_sch (KiCad schematic)
At the start: 86 parts, among them J2 In, J4 18V, J5 Out, Q1 K170, SW1 MuteStompButton, U1 ECC83, U2 ECC83, U3 DC-DC step-down module, U4 DC-DC step-up module, U5 DC-DC step-down module

Commit message: wenzels-fruity-tube-guitar-preamp release-2026-05-r2
Parts:
- removed U5: DC-DC step-down module, Converter_DCDC:Converter_DCDC_Murata_NXExSxxxxMC_SMD, symbol Regulator_Switching:NXE2S1215MC
- added C1, C2: 100n/50V, symbol Device:C
- added C3: 1n/50V, symbol Device:C
- added Q2: K170, symbol Simulation_SPICE:NJFET
- added R33: 1m, symbol Device:R
- added R34: 4k7, symbol Device:R
- added R35: 1k, symbol Device:R
- added R36: 100r, symbol Device:R
- C36: value 470p/50V -> 10n/50V
- U4: Field5 5-12VDC → 300-1200VDC 10mA -> 18VDC → 320VDC/10mA
Connections:
- net VC: now also Q2.1 (D)
- net VCbias: now also R33.1
- net at C23.1, D3.1 (K), J4.2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: now also U4.3 (+VIN)
- net at R14.1, R6.1: now also C3.1, R35.2; no longer J2.T
- new net: J2.T, R36.1
- new net: C2.1, Q2.3 (S), R34.1
- new net: C2.2, R35.1
- new net: C1.1, R36.2
- new net: C1.2, Q2.2 (G), R33.2
- new net: C3.2, R34.2
Other:
- moved on the sheet: C13, C15, C16, C19, C5, C6, J2, R1, R2, R22, R3, U4

Commit message: wenzels-fruity-tube-guitar-preamp release-2026-06-r3
Parts:
- added C14: 15n/400V, symbol Device:C
- added C17, C18, C20, C21: 10u/400V, symbol Device:C_Polarized
- added C4: 100n/50V, symbol Device:C
- added C9: 4700u/25V, symbol Device:C_Polarized
- added D1: 1N5819, Diode_THT:D_DO-41_SOD81_P10.16mm_Horizontal, symbol Diode:1N5819
- added D2: LED, symbol Device:LED
- added J1: 18V SEND, symbol Connector:Jack-DC
- added J3: 320V RECEIVE, symbol Connector:Jack-DC
- added J6: 18V RECEIVE, symbol Connector:Jack-DC
- added J7: 320V SEND, symbol Connector:Jack-DC
- added R37: 2r2, symbol Device:R
- added RLED1: 10k, symbol Device:R
- added SW2: 18V minus to case, Button_Switch_SMD:Nidec_Copal_CAS-120A, symbol Switch:SW_Nidec_CAS-120A1
- added SW3: 320V minus to case, Button_Switch_SMD:Nidec_Copal_CAS-120A, symbol Switch:SW_Nidec_CAS-120A1
Connections:
- net Expected/recommended (adjust U4): 320V: now also J3.1; no longer R3.1, U4.8 (+VOUT)
- net Expected/recommended: 320V: now also R3.1
- net GND: now also C3.2, R34.2, J1.2, J3.2; no longer U4.1 (-VIN), U4.7 (-VOUT)
- net at C23.1, D3.1 (K), J4.2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: now also J1.1; no longer U4.3 (+VIN)
- new net: C4.1, D1.1 (K), J6.1, R37.1, RLED1.1
- new net: C9.1, R37.2, U4.3 (+VIN)
- new net: C14.1, C17.1, C18.1, C20.1, C21.1, J7.1, U4.8 (+VOUT)
- new net: C14.2, C17.2, C18.2, C20.2, C21.2, J7.2, SW3.1 (C), U4.7 (-VOUT)
- new net: C4.2, C9.2, D1.2 (A), D2.1 (K), J6.2, SW2.1 (C), U4.1 (-VIN)
- new net: D2.2 (A), RLED1.2
- new net Enclosure: SW2.2 (B), SW3.2 (B)
- no-connect marks 3 -> 5
Other:
- note added: "External enclosure"
- moved on the sheet: C1, C13, C15, C16, C19, C2, C3, C42, C43, C44, C5, C6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
