File: wenzels-powered-guitar-cabinets/wenzels-powered-guitar-cabinet-2606-bridged-pair.kicad_sch (KiCad schematic)
At the start: 93 parts, among them J1 4Ω secondary, J2 8Ω secondary, J3 16Ω secondary, J6 AC power in, J7 Switching-Mode Power Supply, J8 Input, SW3 GND-1

Commit message: wenzels-powered-guitar-cabinet-2606 r1-wip-2
Parts:
- TR1: Field5 (none) -> Secondary polarity is flipped in order to keep; Field6 (none) -> the signal in phase (each amp is inverting); Field7 (none) -> 1:4 configuration (1:2 for each amp)
Connections:
- net at R16.1, R17.1: now also TR1.14, TR1.B3; no longer TR1.8, TR1.B2
- net at R23.1, R24.1: now also TR1.8, TR1.B2; no longer TR1.14, TR1.B3
Changed lines of the file:
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@@
 		(title "Wenzel’s Powered Guitar Cabinet 2606 (bridged-pair)")
 		(date "June 2026")
-		(rev "r1-wip-1")
+		(rev "r1-wip-2")
 		(company "WORK IN PROGRESS...")
 	)
@@
 	)
 	(junction
-		(at 163.83 236.22)
-		(diameter 0)
-		(color 0 0 0 0)
-	)
-	(junction
 		(at 240.03 269.24)
 		(diameter 0)
@@
 	)
 	(junction
+		(at 163.83 236.22)
+		(diameter 0)
+		(color 0 0 0 0)
+	)
+	(junction
 		(at 53.34 220.98)
 		(diameter 0)
@@
 	(wire
 		(pts
+			(xy 78.74 152.4) (xy 78.74 236.22)
+		)
+		(stroke
+			(width 0)
+			(type default)
+		)
+	)
+	(wire
+		(pts
 			(xy 303.53 203.2) (xy 303.53 205.74)
 		)
@@
 	(wire
 		(pts
-			(xy 55.88 236.22) (xy 58.42 236.22)
+			(xy 163.83 220.98) (xy 163.83 236.22)
 		)
 		(stroke
 			(width 0)
 			(type default)
-			(color 0 0 194 1)
 		)
 	)
 	(wire
 		(pts
-			(xy 361.95 91.44) (xy 361.95 96.52)
+			(xy 55.88 236.22) (xy 58.42 236.22)
 		)
 		(stroke
 			(width 0)
 			(type default)
+			(color 0 0 194 1)
 		)
 	)
 	(wire
 		(pts
-			(xy 102.87 193.04) (xy 107.95 193.04)
+			(xy 361.95 91.44) (xy 361.95 96.52)
 		)
 		(stroke
 			(width 0)
 			(type default)
-			(color 132 132 132 1)
 		)
 	)
 	(wire
 		(pts
-			(xy 236.22 86.36) (xy 238.76 86.36)
+			(xy 102.87 193.04) (xy 107.95 193.04)
 		)
 		(stroke
 			(width 0)
 			(type default)
+			(color 132 132 132 1)
 		)
 	)
 	(wire
 		(pts
-			(xy 270.51 193.04) (xy 274.32 193.04)
+			(xy 236.22 86.36) (xy 238.76 86.36)
 		)
 		(stroke
@@
 	(wire
 		(pts
-			(xy 68.58 236.22) (xy 163.83 236.22)
+			(xy 270.51 193.04) (xy 274.32 193.04)
 		)
 		(stroke
@@
 	(wire
 		(pts
-			(xy 72.39 152.4) (xy 54.61 152.4)
+			(xy 54.61 152.4) (xy 78.74 152.4)
 		)
 		(stroke
@@
 	(wire
 		(pts
-			(xy 68.58 220.98) (xy 72.39 220.98)
+			(xy 68.58 220.98) (xy 163.83 220.98)
 		)
 		(stroke
@@
 	(wire
 		(pts
+			(xy 78.74 236.22) (xy 68.58 236.22)
+		)
+		(stroke
+			(width 0)
+			(type default)
+		)
+	)
+	(wire
+		(pts
 			(xy 252.73 165.1) (xy 252.73 156.21)
 		)
@@
 	(wire
 		(pts
-			(xy 72.39 220.98) (xy 72.39 152.4)
-		)
-		(stroke
-			(width 0)
-			(type default)
-		)
-	)
-	(wire
-		(pts
 			(xy 189.23 86.36) (xy 207.01 86.36)
 		)
@@
 			)
 		)
+		(property "Field5" "Secondary polarity is flipped in order to keep"
+			(at 76.962 204.47 0)
+			(effects
+				(font
+					(size 1.27 1.27)
+				)
+				(justify right)
+			)
+		)
+		(property "Field6" "the signal in phase (each amp is inverting)"
+			(at 76.962 207.264 0)
+			(effects
+				(font
+					(size 1.27 1.27)
+				)
+				(justify right)
+			)
+		)
+		(property "Field7" "1:4 configuration (1:2 for each amp)"
+			(at 76.962 210.058 0)
+			(effects
+				(font
+					(size 1.27 1.27)
+				)
+				(justify right)
+			)
+		)
