File: wenzels-powered-guitar-cabinets/wenzels-powered-guitar-cabinet-2606-bridged-pair.kicad_sch (KiCad schematic)
At the start: 93 parts, among them J1 4Ω secondary, J2 8Ω secondary, J3 16Ω secondary, J6 AC power in, J7 Switching-Mode Power Supply, J8 Input, SW3 GND-1

Commit message: powered-guitar-cabinet 2606 bridged-pair r1-wip-3
Parts:
- removed C2, C20: 2200u, symbol Device:C_Polarized
- C1, C19: value 2200u -> 680u
- OT1: Field6 100W RMS, 45Hz–20kHz -> 100W RMS, 40Hz–20kHz
Connections:
- net at OT1.2 (4Ω), R6.1: now also C1.2
- net at OT1.1 (0Ω), R41.1: now also C19.2
Other:
- note added: "C1 and C19, their values and polarity rely on: - It’s a bridge pair (so that they are kind of unpolarized in the pair) - Emitter and output resistor values - 4 ohms load seen from the output transformer To set the cut-off frequency to around 45Hz to match the output transformer bottom frequency."
- moved on the sheet: R41, R6
