File: wenzels-powered-guitar-cabinets/wenzels-powered-guitar-cabinet-2606-single-amp-hifi-ish.kicad_sch (KiCad schematic)
At the start: 49 parts, among them J1 8Ω min, J2 Input, J6 AC power in, J7 Switching-Mode Power Supply, SW3 GND-LIFT

Commit message: 2606-single-amp-hifi-ish r1-wip-2 add biasing info text
Other:
- note added: "Biasing the amp: Start with bias trimmer R8 set to minimum resistance. Power up with no load first, input shorted to ground. Measure DC millivolts across R1 and R2. Because R1 and R2 are 0.22Ω: 11mV ≈ 50mA 15mV ≈ 68mA 18mV ≈ 82mA 22mV ≈ 100mA Aim for about 12mV-18mV across each resistor. A good starting target is 15mV. Let the amp warm up for 10-15 minutes. Measure again and adjust if needed."
Changed lines of the file:
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@@
+		)
+	)
+	(text "Biasing the amp:\n\nStart with bias trimmer R8 set to minimum resistance.\nPower up with no load first, input shorted to ground.\n\nMeasure DC millivolts across R1 and R2.\nBecause R1 and R2 are 0.22Ω:\n\n11mV ≈ 50mA\n15mV ≈ 68mA\n18mV ≈ 82mA\n22mV ≈ 100mA\n\nAim for about 12mV-18mV across each resistor.\nA good starting target is 15mV.\n\nLet the amp warm up for 10-15 minutes.\nMeasure again and adjust if needed."
+		(exclude_from_sim no)
+		(at 25.654 25.4 0)
+		(effects
+			(font
+				(size 1.27 1.27)
+			)
+			(justify left top)
 		)
 	)
