File: wenzels-powered-guitar-cabinets/wenzels-powered-guitar-cabinet-2606-single-amp.kicad_sch (KiCad schematic)
At the start: 48 parts, among them J1 4Ω secondary, J2 8Ω secondary, J3 16Ω secondary, J4 Input

Commit message: wenzels-powered-guitar-cabinet 2606-single-amp r1-wip-4
Remove bridged-pair because new designed is intended to use single-ended
for the 100W-class power into 8Ω load. Bridge-mode is no longer
necessary to deliver enough power.

Also remove HiFi-ish version for now as it needs re-adjustments.
Maybe later I’ll make an updated version.
Parts:
- removed C9: 100p, symbol Device:C
- added C12, C13, C14, C9: 200u, symbol Device:C_Polarized
- added C15: 82n, symbol Device:C
- added C16, C17, C18, C22, C24: 100n, symbol Device:C
- added C19: 220u, symbol Device:C_Polarized
- added C20: 10n, symbol Device:C
- added C21, C23: 470u, symbol Device:C_Polarized
- added J5, J6: 8Ω primary, symbol Connector_Audio:AudioJack2
- added J7: 8Ω feedback source, symbol Connector_Audio:AudioJack2
- added J8: 8Ω feedback source pass-through, symbol Connector_Audio:AudioJack2
- added Q1, Q2: MPSA42, Package_TO_SOT_THT:TO-92_Inline, symbol Transistor_BJT:MPSA42
- added R23: 56k, symbol Device:R
- added R24: 12k, symbol Device:R
- added R25: 330, symbol Device:R
- added R26, R28: 10k, symbol Device:R
- added R27, R30: 1k, symbol Device:R
- added R29: 100, symbol Device:R
- C1, C2: value 2200u -> 200u
- C10, C11: value 2200u -> 10000u
- OT1: Field6 100W RMS, 45Hz–20kHz -> 100W RMS, 40Hz–20kHz
- R17: value 47k -> 470k
- R18, R19: value 47k -> 22k
- R20, R21: value 2r -> 0.5; Field5 100W -> 25W
- R22: value 470r -> 100k; Field5 5W -> (none); Field6 OT no load protection -> (none)
- R3: value 2r -> 0.25; Field5 100W -> 25W
- R6: value 4k7 -> 10k; Field5 1W -> (none)
Connections:
- net GND: now also C16.2, C17.1, C18.2, C19.2, C20.2, C21.2, C22.2, C23.1, C24.2, J6.S, J7.S, J8.S, R23.2, R26.2, R28.2; no longer OT1.1 (0Ω)
- net VCC: now also C16.1, C21.1, C22.1, R25.1
- net VEE: now also C17.2, C23.2, C24.1
- net at C2.1, R6.1: now also C12.1, C14.1, J6.T; no longer OT1.2 (4Ω)
- net at C1.2, C2.2: now also C12.2, C13.2, C14.2, C9.2
- net at J1.S, J2.S, J3.S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: no longer R22.2
- net at J1.T, OT1.5 (4Ω): no longer R18.2, R22.1
- net at C7.2, D1.1 (K), Qvas.2 (B)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: now also R30.2; no longer C3.2
- net at C6.1, R16.2: now also C15.1; no longer C3.1
- net at C1.1, R3.2: now also C13.1, C9.1
- net at OT1.3 (8Ω): now also J5.T
- new net: C18.1, C19.1, Q2.3 (C), R22.1, R24.1, R25.2
- new net: C15.2, Q1.2 (B), R22.2, R23.1
- new net: J7.T, J8.T, R18.2
- new net: Q1.3 (C), R24.2, R27.1
- new net: Q2.1 (E), R28.1, R29.1
- new net: C20.1, C3.1, R29.2
- new net: J5.S, OT1.1 (0Ω)
- new net: C3.2, R30.1
- new net: Q2.2 (B), R27.2
- new net: Q1.1 (E), R26.1
Other:
- note added: "Aiming for 280u-300u total capacitance. Into 8 ohms load it’s calculated close to 60Hz cut-off (not only bass reduction but actually making low end progressively looser, so damping factor drops more the lower it goes). Parallel caps are better in order to distribute current handling demand, and not depend too much on the high current ripple ratings for the caps."
- note added: "Biasing: Start with bias trimmer R8 set to minimum resistance. Power up with no load first: transformer disconnected, input shorted to ground, and current limiting if available. Measure DC millivolts across R1 and R2. Because R1 and R2 are 1Ω, 1mV = 1mA. Aim for 50mV-80mV across each resistor. Let the amp warm up for 10-15 minutes. Measure again and adjust if needed. Start with minimum, 50mV. The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"
- note added: "Input inverting stage (to make the amp in-phase relative to the input). And also tone shaping (high-pass set to around 55Hz at input)."
- note added: "LF VOICING: ~55 Hz input HPF + ~57-60 Hz passive output-coupling pole are cascaded, so total electrical LF rolloff starts higher than either pole alone. Exact response varies somewhat with NFB setting. Despite this, LF damping falls strongly with frequency because of the series output capacitor. Speaker/cab resonances therefore have more influence, so perceived bass can remain strong and "bloomin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"
- note added: "Make sure R25 pulse rating is sufficient to handle the surge current at startup, when the caps are charging."
- note added: "Make sure that the transformer secondary polarity is in-phase with the primary. The first signal test should be made with the NFB pot at maximum resistance (minimum pot position). Then reduce resistance gradually (turn the pot clockwise). If gain increases, the amp becomes unstable, or it howls as feedback is increased, the feedback-secondary polarity is wrong and the two feedback wires must be r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"
- note added: "R20/R21 must have adequate pulse-energy/inrush capability. Each rail charges 10,000 µF at startup (~15.7 J stored per rail at 56 V). Use pulse-rated wirewound/chassis resistors and/or current-limited/soft-start supply."
- note removed: "Biasing: Start with bias trimmer R8 set to minimum resistance. Power up with no load first: transformer disconnected, input shorted to ground, and current limiting if available. Measure DC millivolts across R1 and R2. Because R1 and R2 are 1Ω, 1mV = 1mA. Aim for 50mV-80mV across each resistor. Let the amp warm up for 10-15 minutes. Measure again and adjust if needed. Negative feedback (NFB pot): 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"
- note removed: "This is my own discrete Class AB amplifier design with MOSFET push-pull output stage intended for guitar amplification. It is relatively simple and straightforward. I intentionally avoided any HiFi-tweaks (like differential input, "current source", "current mirror" or whatever, I only used Vbe multiplier here to bias the MOSFETs), the amp is intended to be imperfect, having damping factor less th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"
- moved on the sheet: C10, C11, C3, C4, C5, C7, C8, D1, D2, D3, D4, D5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
