File: wenzels-powered-guitar-cabinets/wenzels-powered-guitar-cabinet-2610.kicad_sch (KiCad schematic)
At the start: 44 parts, among them J1 AC power in, J13 4Ω secondary 1, J14 8Ω secondary 1, J15 16Ω secondary 1, J16 4Ω output 1, J17 4Ω primary, J2 In 1, J4 Switching-Mode Power Supply, U2 TDA7294

Commit message: wenzels-powered-guitar-cabinet-2610 release-2610-power-amplifier-2026-10-r1
Parts:
- added C26, C42, C58: 33n, symbol Device:C
- added C27, C43, C59: 100p, symbol Device:C
- added C28, C29, C37, C44, C45, C53, C60, C61, C69: 100n, symbol Device:C
- added C30, C31, C46, C47, C62, C63: 470u, symbol Device:C_Polarized
- added C32, C48, C64: 15u, symbol Device:C_Polarized
- added C33, C34, C36, C49, C50, C52, C65, C66, C68: 22u, symbol Device:C_Polarized
- added C35, C51, C67: 10p, symbol Device:C
- added C38, C39, C40, C41, C54, C55, C56, C57, C70, C71, C72, C73: 680u, symbol Device:C_Polarized
- added D3, D4, D5: 1N4148, Diode_THT:D_DO-35_SOD27_P7.62mm_Horizontal, symbol Diode:1N4148
- added J18: 4Ω output 2, symbol Connector_Audio:AudioJack2
- added J19: 4Ω primary 2, symbol Connector_Audio:AudioJack2
- added J20: 4Ω secondary 2, symbol Connector_Audio:AudioJack2
- added J21: 8Ω secondary 2, symbol Connector_Audio:AudioJack2
- added J22: 16Ω secondary 2, symbol Connector_Audio:AudioJack2
- added J23: 4Ω output 3, symbol Connector_Audio:AudioJack2
- added J24: 4Ω primary 3, symbol Connector_Audio:AudioJack2
- added J25: 4Ω secondary 3, symbol Connector_Audio:AudioJack2
- added J26: 8Ω secondary 3, symbol Connector_Audio:AudioJack2
- added J27: 16Ω secondary 3, symbol Connector_Audio:AudioJack2
- added J28: 4Ω output 4, symbol Connector_Audio:AudioJack2
- added J29: 4Ω primary 4, symbol Connector_Audio:AudioJack2
- added J3: In 2, symbol Connector_Audio:AudioJack3_Switch
- added J30: 4Ω secondary 4, symbol Connector_Audio:AudioJack2
- added J31: 8Ω secondary 4, symbol Connector_Audio:AudioJack2
- added J32: 16Ω secondary 4, symbol Connector_Audio:AudioJack2
- added J5: In 3, symbol Connector_Audio:AudioJack3_Switch
- added J6: In 4, symbol Connector_Audio:AudioJack3_Switch
- added L3, L4, L5: 5uH, symbol Device:L
- added R19, R29, R40: 68k, symbol Device:R
- added R20, R23, R30, R33, R41, R44: 30k, symbol Device:R
- added R21, R31, R42: 330, symbol Device:R
- added R22, R28, R32, R39, R43, R50: 10k, symbol Device:R
- added R24, R25, R34, R35, R45, R46: 22k, symbol Device:R
- added R26, R37, R48: 2.7r, symbol Device:R
- added R27, R38, R49: 0.5, symbol Device:R
- added R36, R47, R9: 10, symbol Device:R
- added TR2, TR3, TR4: Impedance transformer, symbol Transformer:TRANSF4
- added U3, U4, U5: TDA7294, Package_TO_SOT_THT:TO-220-15_P2.54x2.54mm_StaggerOdd_Lead4.58mm_Vertical, symbol Amplifier_Audio:TDA7294
- J17: value 4Ω primary -> 4Ω primary 1
- J4: Field5 ±24V to ±40V / 500W -> ±24V to ±29V / 500W
Connections:
- net GND: now also C27.2, C28.2, C29.2, C30.2, C31.1, C32.2, C33.2, C34.2, C37.2, C43.2, C44.2, C45.2, C46.2, C47.1, C48.2, C49.2, C50.2, C53.2, C59.2, C60.2, C61.2, C62.2, C63.1, C64.2, C65.2, C66.2, C69.2, J18.S, J23.S, J28.S, J3.R, J3.RN, J3.S, J3.SN, J3.TN, J5.R, J5.RN, J5.S, J5.SN, J5.TN, J6.R, J6.RN, J6.S, J6.SN, J6.TN, R20.2, R28.2, R30.2, R39.2, R41.2, R50.2, U3.1 (SGND), U3.4 (SIG_GND), U4.1 (SGND), U4.4 (SIG_GND), U5.1 (SGND), U5.4 (SIG_GND)
- net V+: now also C28.1, C30.1, C44.1, C46.1, C60.1, C62.1, D3.1 (K), D4.1 (K), D5.1 (K), R23.2, R24.1, R33.2, R34.1, R44.2, R45.1, U3.13 (+Vs), U3.7 (+Vs), U4.13 (+Vs), U4.7 (+Vs), U5.13 (+Vs), U5.7 (+Vs)
- net V-: now also C29.1, C31.2, C45.1, C47.2, C61.1, C63.2, U3.15 (-Vs), U3.8 (-Vs), U4.15 (-Vs), U4.8 (-Vs), U5.15 (-Vs), U5.8 (-Vs)
- new net: C50.1, R34.2, U4.9 (STBY)
- new net: C68.1, U5.6 (BOOT)
- new net: C67.2, C68.2, L5.1, R46.1, R47.2, U5.14
- new net: C49.1, R32.2, U4.10 (MUTE)
- new net: C51.2, C52.2, L4.1, R35.1, R36.2, U4.14
- new net: C51.1, R31.1, R35.2, U4.2 (-)
- new net: C42.2, C43.1, R30.1, U4.3 (+)
- new net: C52.1, U4.6 (BOOT)
- new net: L3.2, R26.1, R27.1, R9.1
- new net: C38.1, C39.1, R27.2
- new net: J25.S, J26.S, J26.T, J27.S, TR3.4 (0Ω), TR3.6 (8Ω)
- new net: J27.T, TR3.7 (16Ω)
- new net: C48.1, R31.2
- new net: D5.2 (A), R43.1, R44.1
- new net: L5.2, R47.1, R48.1, R49.1
- new net: C69.1, R48.2
- new net: L4.2, R36.1, R37.1, R38.1
- new net: C54.1, C55.1, R38.2
- new net: C35.2, C36.2, L3.1, R25.1, R9.2, U3.14
- new net: J24.S, TR3.1 (0Ω)
- new net: J24.T, TR3.2 (4Ω)
- new net: C70.1, C71.1, R49.2
- new net: C70.2, C71.2, C72.2, C73.2
- new net: C37.1, R26.2
- new net: J3.T, R19.2
- new net: C35.1, R21.1, R25.2, U3.2 (-)
- new net: J30.S, J31.S, J31.T, J32.S, TR4.4 (0Ω), TR4.6 (8Ω)
- new net: J30.T, TR4.5 (4Ω)
- new net: J20.S, J21.S, J21.T, J22.S, TR2.4 (0Ω), TR2.6 (8Ω)
- new net: J22.T, TR2.7 (16Ω)
- new net: J6.T, R40.2
- new net: C67.1, R42.1, R46.2, U5.2 (-)
- new net: C64.1, R42.2
- new net: J32.T, TR4.7 (16Ω)
- new net: J29.S, TR4.1 (0Ω)
- new net: J29.T, TR4.2 (4Ω)
- new net: D3.2 (A), R22.1, R23.1
- new net: C33.1, R22.2, U3.10 (MUTE)
- new net: C56.1, C57.1, J23.T, R39.1
- new net: C72.1, C73.1, J28.T, R50.1
- new net: C26.1, R19.1
- new net: C26.2, C27.1, R20.1, U3.3 (+)
- new net: C54.2, C55.2, C56.2, C57.2
- new net: J25.T, TR3.5 (4Ω)
- new net: C34.1, R24.2, U3.9 (STBY)
- new net: C65.1, R43.2, U5.10 (MUTE)
- new net: C58.2, C59.1, R41.1, U5.3 (+)
- new net: C66.1, R45.2, U5.9 (STBY)
- new net: C40.1, C41.1, J18.T, R28.1
- new net: C38.2, C39.2, C40.2, C41.2
- new net: C32.1, R21.2
- new net: D4.2 (A), R32.1, R33.1
- new net: C36.1, U3.6 (BOOT)
- new net: C58.1, R40.1
- new net: C42.1, R29.1
- new net: J5.T, R29.2
- new net: J20.T, TR2.5 (4Ω)
- new net: C53.1, R37.2
- new net: J19.S, TR2.1 (0Ω)
- new net: J19.T, TR2.2 (4Ω)
- no-connect marks 1 -> 4
Other:
- note added: "40W-50W of power for each amplifier channel at ±24V supply into 4 ohms (as “seen” by the amplifier, you can connect 8 or 16 ohms cab/speaker into the respective transformer secondary port, so that for the amplifier it stays 4 ohms load). In my experience it’s enough to power 2x12/4x12 cab with just one channel at ±24V supply. Everything is designed around 4 ohms load. The impedance transformers a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"
- note added: "Aiming for 600-680 total capacitance for around 50-60Hz cut-off. Note that it does not mean low frequencies will be perceived significantly lower. The damping factor below the cut-off is significantly reduced, which would create more low end “bloom”, and more perceivable deepness. More caps are better to distribute current (make sure ESR is consistent so some caps are not overworking over others)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"
- note added: "The power amp IC are all TDA7294"
- note removed: "--------------TODO----------------- You should expect around 30W of power for each amplifier channel into 4 ohms. The idea is that all 4 are driving 4 speakers independently, so that you get enough power, while each individual amps is not that powerful. Everything is designed around 4 ohms load. The impedance transformers are supposed to keep that 4 ohms load consistency regardless of actual spea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"
- note removed: "Aiming for 680-700uF total capacitance for around 50Hz cut-off. Note that it does not mean low frequencies will be perceived significantly lower. The damping factor below the cut-off is significantly reduced, which would create more low end “bloom”, and more perceivable deepness. More caps are better to distribute current (make sure ESR is consistent so some caps are not overworking over others).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"
- note removed: "Each cap ≥1.5 A @100 Hz. Verify LF frequency derating."
- title: Wenzel’s Powered Guitar Cabinet 2610 -> Wenzel’s Guitar Power Amplifier 2610
- moved on the sheet: C10, C11, C12, C13, C14, C15, C16, C17, C18, C19, C20, C21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
