File: wenzels-tubinizer/wenzels-tubinizer.kicad_sch (KiCad schematic)
At the start: 125 parts, among them J1 18V, J2 Input-L, J3 Output-L, J4 Input-R, J5 Output-R, SW1 GND-LIFT, SW2 GND-LIFT, SW3 GND-LIFT, SW4 GND-LIFT, U1 DC-DC step-down module, U1 ECC83, U2 DC-DC step-up module, U3 DC-DC step-up module, U4 TL072, U5 TL072, U6 TL072

Commit message: wenzels-tubinizer release-2026-08-r1
Parts:
- removed C1: 2200u/25V, symbol Device:C_Polarized
- removed C12, C15, C34, C37: 4u7/50V, symbol Device:C_Polarized
- removed C16, C32, C45, C46: 47u/50V, symbol Device:C_Polarized
- removed C23: 100n/50V, symbol Device:C
- removed C51, C52, C53: 100n, symbol Device:C
- removed D3: 1N5819, Diode_THT:D_DO-41_SOD81_P10.16mm_Horizontal, symbol Diode:1N5819
- removed D4: LED, symbol Device:LED
- removed J1: 18V, symbol Connector:Jack-DC
- removed R10, R12, R13, R29, R31, R50, R51, R9: 220k, symbol Device:R
- removed R18: 22k, symbol Device:R
- removed R8: 2r2/1W, symbol Device:R
- removed RLED2: 10k, symbol Device:R
- removed U3: DC-DC step-up module, Converter_DCDC:Converter_DCDC_Murata_NXExSxxxxMC_SMD, symbol Regulator_Switching:NXE2S1215MC
- removed unit 3 of U4
- removed unit 3 of U5
- removed unit 3 of U6
- added C12, C15, C16: 100n/50V, symbol Device:C
- added C18: 100u/50V, symbol Device:C_Polarized
- added C20, C21, C23: 10u/400V, symbol Device:C_Polarized
- added C32, C34, C37, C45, C46: 100n, symbol Device:C
- added J1: IEC_60320_C14_Receptacle, symbol Connector:IEC_60320_C14_Receptacle
- added U1: TL072, symbol Amplifier_Operational:TL072
- added unit 3 of U2
- added unit 3 of U3
- added U4: TMLM04112, Converter_ACDC:Converter_ACDC_TRACO_TMLM-04_THT, symbol Converter_ACDC:TMLM04112
- added U5: RAC20-12DK, Converter_ACDC:Converter_ACDC_Recom_RAC20-xxDK_THT, symbol Converter_ACDC:RAC20-12DK
- C25, C29: value 4u7/50V -> 10u/400V
- C31: value 47u/50V -> 10u/400V
- C50: Field5 50V -> >=63V
- R15: value 47r -> 100r
- R17: value 22k -> 100r
- U1: Field5 Adjustable 18VDC → ≈12VDC 3A -> Adjustable 15VDC → ≈12VDC 3A
- U2: Field5 18VDC → 320VDC/10mA -> 12-24VDC → 200-450VDC
- renumbered U4 to U1, U5 to U2, U6 to U3
Connections:
- net Grounded  is gone; now on net GND: C2.2, C26.2, C30.2, C33.2, C41.2, C47.2, C48.2, C49.2, R11.2, R52.2, SW2.1, SW4.1, Volume-L.1, Volume-R.1
- net GND: now also C25.2, C27.1, C29.2, C31.2, C36.1, R21.2, R26.2, R34.2, R45.2, U2.5 (+), U3.5 (+), C12.2, C15.1, C16.1, C18.1, C20.2, C21.2, C23.2, C32.1, C34.2, C37.1, C45.2, C46.1, U5.4 (Com); no longer C9.2, U2.1 (-VIN)
- net VA: now also C29.1, C20.1, C23.1
- net VB: now also C25.1, C31.1, R1.1, C21.1; no longer R1.2
- net at C36.2, R34.1, U1.5 (+): now also R33.2
- net at C35.2, R35.1, U1.6 (-): now also R32.2; no longer C29.1
- net at C35.1, R35.2, U1.7: now also R36.1
- net at R46.2, U3.1, U3.2 (-): now also R48.1
- net at R37.1: now also U4.2 (Vout+); no longer U1.3 (+VIN)
- net at R47.2, U3.7: now also R49.1
- net at C24.1, R20.2, U1.1: now also R19.1
- net at C24.2, R20.1, U1.2 (-): now also R16.2
- net at C27.2, R21.1, U1.3 (+): now also R23.2; no longer C25.1
- net at R24.2, U2.7: now also R27.1; no longer C31.1
- net at R25.2, U2.1, U2.2 (-): now also R28.1
- net +15V: now reaches R15.1
- net +15V: now also U1.3 (+VIN), C12.1, U5.5 (+Vout)
- net Adjust U2 to 320V here renamed Adjust U2 to 300V here
- net Adjust U2 to 300V here: now also R1.2; no longer R1.1
- net Adjust U3 to 30–33V here (30V is more safe conservative value for TL072): no longer names the net of C4.1, C7.1, R15.2
- net Adjust U3 to 30–33V here (30V is more safe conservative value for TL072): now also C32.2, C37.2, C46.2, U1.8 (V+), U2.8 (V+), U3.8 (V+); no longer C50.1, R17.2
- removed net Vref: C27.1, C36.1, R17.1, R21.2, R26.2, R34.2, R45.2, U2.5 (+), U3.5 (+)
- new net: C16.2, C18.2, C34.1, C45.1, C50.1, R17.1, U1.4 (V-), U2.4 (V-), U3.4 (V-)
- new net: C9.2, U2.1 (-VIN), U4.3 (Vout-)
- new net: J1.1 (L), U4.5 (AC(L)), U5.2 (AC(L))
- new net: J1.2 (N), U4.6 (AC(N)), U5.1 (AC(N))
- new net -15V: C15.2, R17.2, U5.3 (-Vout)
- new net Case shield: J1.3 (PE)
Other:
- note added: "Input polarity is flipped (tip goes to inverting input). It helps to restore phase polarity, because the tube gain stage flips the phase too."
- note added: "Technically you can feed the HV booster from the +15V of U5 and U4 would be not necessary then, but in my case U5 was going into overload protection, it doesn’t have enough current capability to handle it. So I had to add U4."
- note removed: "Input polarity is flipped. It helps to restore phase polarity, because the tube gain stage flips the phase too."
- moved on the sheet: C13, C14, C17, C19, C4, C40, C42, C43, C5, C6, C7, C9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
