File: wenzels-real-fuzz-muff-mod/real-fuzz-muff-mod.kicad_sch (KiCad schematic)
At the start: 109 parts, among them J1 Input jack, J2 Output jack, J3 18V, Q1 J113, Q2 J113, Q3 J113, Q4 J113, SW1 CLIP1, SW2 CLIP2, T1 2n2369a, T2 2n2369a, T3 2n2369a, T4 2n2369a

Commit message: wenzels-real-fuzz-muff-mod release-2026-08-r3
Parts:
- removed C21, C31, C32: 47u, electrolytic, symbol Device:C_Polarized
- removed C30: 100n, film, symbol Device:C
- removed D10, D7: BLUE, symbol Device:LED
- removed D8, D9: ORANGE, symbol Device:LED
- removed Q1, Q2, Q3, Q4: J113, Package_TO_SOT_SMD:SOT-23, symbol Transistor_FET:MMBFJ113
- removed R36, R40: 1M, symbol Device:R
- removed R44: 100R, symbol Device:R
- added C21: 100n, film, symbol Device:C
- added C30: 100u, electrolytic, symbol Device:C_Polarized
- added C37: 47u, electrolytic, symbol Device:C_Polarized
- added D7: 39V/1.3W, Diode_SMD:D_MiniMELF, symbol Diode:BZV55B39
- added Q1, Q2, Q3, Q4: 2N3904, Package_TO_SOT_THT:TO-92_Inline, symbol Transistor_BJT:2N3904
- added QC1, QC2, QC3, QC4: BS170, symbol Device:Q_NMOS
- added R28: 100R, symbol Device:R
- added R45, R46: 47k, symbol Device:R
- C14, C20: value 47u -> 100u
- C29: value 100p -> 10n
- J3: value 18V -> 18V-36V
- R27, R31: value 2k -> 1k
- R35, R39: value 1M -> 470k
- T1: Field5 hFE -> (none); Field6 40-60 -> (none); Field7 (none) -> hFE; Field8 (none) -> 40–60
- T2, T3, T4: Field5 hFE 40-60 -> (none); Field7 (none) -> hFE; Field8 (none) -> 40–60
Connections:
- net 18V: now also C21.1, C30.1, D7.1 (K), Q1.3 (C), Q2.3 (C), Q3.3 (C), Q4.3 (C), R28.2, R45.1; no longer C19.1, C20.1, R25.2, R35.1, R39.1
- net GND: now also C21.2, C30.2, C37.2, D7.2 (A), R46.2
- net at R33.1: now also Q2.1 (E)
- net at R30.2, VOLTS2.1: now also Q2.2 (B)
- net at C9.1, R12.2, R13.1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: now also QC3.D, QC3.G
- net at C6.1, R7.2, R8.1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: now also QC1.D, QC1.G
- net at SW2.2 (B), SW2.3 (A): now also QC4.D, QC4.G
- net at R26.2, VOLTS1.1: now also Q1.2 (B)
- net at SW1.2 (B), SW1.3 (A): now also QC2.D, QC2.G
- net at C26.1, R37.1: now also Q3.1 (E)
- net at R29.1: now also Q1.1 (E)
- net at C28.1, R41.1: now also Q4.1 (E)
- net at C28.2, R39.2: now also Q4.2 (B)
- net at C25.2, R35.2: now also Q3.2 (B)
- net 3V-18V renamed 3V-36V
- new net: QC1.S, QC2.S
- new net: C19.1, C20.1, R25.2, R28.1
- new net: QC3.S, QC4.S
- new net: C37.1, R35.1, R39.1, R45.2, R46.1
Other:
- note added: "Check your BS170s pinouts first! They may vary a lot. Don’t just google it, use for example a transistor tester instead."
- note added: "Optional: After cutting the traces you can tap the spot on the PCB where you made a cut with a nail polish to avoid metal corrosion. Or you can avoid cutting the traces by not soldering top ends of R10 and R15, instead wiring them to the extension board."
- note added: "This mod: 1. Removes clipping diodes completely, letting the transistors clip instead, making classic Muff circuit loud and wild, more dynamic, like a real fuzz pedal. At the same time it provides optional/switchable BS170 MOSFET pairs as clipping diodes replacement. The forward voltage is much higher, ≈2.60V (for each direction) vs. ≈0.7V for regular 1n4841. So even though there's no make-up gai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"
- note removed: "LEDs forward voltage measurements RED - 1.93V GREEN - 2.02V BLUE - 2.63V ORANGE - 1.97V YELLOW - 2.10V WHITE - 2.73V"
- note removed: "Optional: After cutting the traces you can tap the spot on the PCB where you made a cut with a nail polish to avoid metal corrosion."
- note removed: "This mod: 1. Removes clipping diodes completely, letting the transistors clip instead, making classic Muff circuit loud and wild, like a real fuzz pedal. 2. Re-routes T4 gain stage to go after T1, giving the clipping stages more pre-gain as they require much more to really clip, since there are no diodes, only transistors clipping when they can amplify no more. And you don't need the final VOLUME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"
- moved on the sheet: SW2
