File: wenzels-real-fuzz-muff-mod/real-fuzz-muff-mod.kicad_sch (KiCad schematic)
At the start: 105 parts, among them J1 Input jack, J2 Output jack, J3 9V-18V, Q1 2N3904, Q2 2N3904, Q3 2N3904, Q4 2N3904, T1 2n2369a, T2 2n2369a, T3 2n2369a, T4 2n2369a

Commit message: wenzels-real-fuzz-muff-mod release-2026-09-r5
Parts:
- removed C28: 1u, electrolytic/film, symbol Device:C_Polarized
- removed J1: Input jack, symbol Connector_Audio:AudioJack2_Switch
- removed J2: Output jack, symbol Connector_Audio:AudioJack2
- removed Q1, Q2, Q3, Q4: 2N3904, Package_TO_SOT_THT:TO-92_Inline, symbol Transistor_BJT:2N3904
- added C26: 100n, ceramic, symbol Device:C
- added C39, C40: 100u, electrolytic, symbol Device:C_Polarized
- added C41, C42, C44, C46: 100n, film, symbol Device:C
- added C43: 68n, film, symbol Device:C
- added C45, C50: 10n, ceramic, symbol Device:C
- added C47: 1n, ceramic, symbol Device:C
- added C49, C52, C55: 220n, film, symbol Device:C
- added C51, C53, C54, C56: 1u, electrolytic, symbol Device:C_Polarized
- added CLEAN: A10k, symbol Device:R_Potentiometer
- added J1: In, symbol Connector:Conn_Coaxial
- added J2: Out, symbol Connector:Conn_Coaxial
- added Q1, Q2: J113, Package_TO_SOT_SMD:SOT-23, symbol Transistor_FET:MMBFJ113
- added R36, R40: 47, symbol Device:R
- added R44, R47, R56: 10k, symbol Device:R
- added R48, R49, R50, R52, R53: 100k, symbol Device:R
- added R51, R57: 100R, symbol Device:R
- added R54: 1k, symbol Device:R
- added R55: 47k, symbol Device:R
- added R58: 2M2, symbol Device:R
- added STARVE-1, STARVE-2: SW_SPDT, symbol Switch:SW_SPDT
- added TIGHT: C100k, symbol Device:R_Potentiometer
- added U1, U2 (x2), U3: TL072, symbol Amplifier_Operational:TL072
- C15: value 10p -> 100p
- C28: footprint film -> ceramic
- C29: value 10n -> 100n
- R27: value 2k -> 1k
- R31: value 2k -> 10k
- R32: value 10 -> 47
- R33: value 47 -> 1k
- R35: value 470k -> 2M2
- R37: value 10k -> 47k
- R39: value 220k -> 47k
- R41: value 10k -> 100R
- R42: value 100R -> 2M2
- R43: value 100k -> 470k
Connections:
- net GND: now also C28.2, R33.2, C26.2, C39.2, C40.2, C44.2, C45.2, C47.2, C50.2, C56.2, CLEAN.1, J1.2 (Ext), J2.2 (Ext), R47.2, R52.2, R58.2, U1.4 (V-), U2.4 (V-), U3.4 (V-); no longer R31.2, R37.2, R41.2, R43.2
- net at R1.1, R23.1: now also R41.2, R54.1
- net at R41.1: now also C51.2
- net at R39.2: now also R37.1, U1.6 (-); no longer C28.2
- net at C21.1, C30.1, R26.1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: now also C28.1, C29.1, R31.1, C26.1, Q1.1 (D), Q2.1 (D), R36.1, U1.8 (V+), U2.8 (V+), U3.8 (V+); no longer R30.1
- net at R34.1: now also J1.1 (In), R58.1; no longer Volume.2
- net at C32.1, R26.2, VOLTS1.1: now also Q1.3 (G), STARVE-1.1 (A)
- net at R42.1: now also C41.2, U2.3 (+)
- net at C37.1, R45.2, R46.1: now also R35.2, R42.2, R43.2, C44.1, R53.2, U1.5 (+), U3.5 (+); no longer R35.1, R39.1
- net at C27.1, TAME.2, TAME.3: now also C41.1; no longer C28.1
- net at R27.1, VOLTS1.2, VOLTS1.3: now also R30.2
- net at C38.1, VOLTS2.1: now also R31.2, Q2.3 (G), STARVE-2.1 (A); no longer R30.2
- net at VOLTS2.2, VOLTS2.3: now also R33.1, R44.2; no longer R31.1
- net at R29.1: now also Q1.2 (S)
- net at C25.2: now also R35.1, U1.3 (+); no longer R35.2
- net at R38.1: now also U2.1, U2.2 (-); no longer R37.1
- net ≈3V–≈18V (for 18V supply): no longer names the net of C31.1, R10.1, R29.2
- net ≈3V–≈18V (for 18V supply): no longer C23.1, R15.1, R33.2
- net ≈9V–≈18V: no longer names the net of R20.1, R21.1, R32.2
- net ≈9V–≈18V: now also C39.1; no longer C14.1, R4.1
- new net: C49.2, R50.1
- new net: R48.1, R49.2, R50.2, U3.6 (-)
- new net: C45.1, J2.1 (In), R51.2, R52.1
- new net: C50.1, CLEAN.3, R57.2
- new net: C56.1, R56.1
- new net: C46.1, C47.1, R54.2
- new net: C55.2, R49.1
- new net: C49.1, CLEAN.2
- new net: R44.1, STARVE-2.2 (B)
- new net: C52.1, U1.1, U1.2 (-)
- new net: C52.2, R39.1
- new net: C42.1, Volume.2
- new net: C23.1, R15.1, R40.2
- new net: R47.1, TIGHT.3
- new net: C40.1, R36.2, R4.1
- new net: C53.2, R57.1
- new net: C42.2, R43.1, U2.3 (+)
- new net: C54.1, R48.2, U3.7
- new net: R30.1, STARVE-1.2 (B)
- new net: C51.1, R37.2, U1.7
- new net: C53.1, R55.2, U3.1
- new net: C46.2, R53.1, U3.3 (+)
- new net: C43.2, C55.1, TIGHT.1, TIGHT.2
- new net: C43.1, U2.1, U2.2 (-)
- new net: R55.1, R56.2, U3.2 (-)
- new net: Q2.2 (S), R40.1
- new net: C54.2, R51.1
- new net No connection to power supply rail: C14.1
- no-connect marks 20 -> 28
Other:
- note added: "C14, C5 and C8 are not needed (you don’t need to solder them on)"
- note added: "Do not solder top ends of R4, R10, R15, R20, R21. Instead wire them to the extension board as shown."
- note added: "TAME ≈ 21.95 kHz → 495 Hz TIGHT ≈ 49 Hz → 258 Hz"
- note added: "VOLTS1 and VOLTS2 are ranging: - ≈1.5V-≈18V (for 18V supply) - ≈0.8V-≈9V (for 9V supply) With STARVE switch engaged: - ≈1.5V-≈9V (for 18V supply) - ≈0.8V-≈4.5V (for 9V supply)"
- note added: "Will work at 9V, but headroom will be reduced. Clean blend may clip on strong transients. 18V recommended."
- note removed: "C5 and C8 are not needed (you don’t need to solder them on)"
- note removed: "Cut the trace using a scalpel"
- note removed: "Optional: After cutting the traces you can tap the spot on the PCB where you made a cut with a nail polish to avoid metal corrosion. Or you can avoid cutting the traces by not soldering top ends of R10 and R15, instead wiring them to the extension board."
- moved on the sheet: C27, C31, C32, C37, R26, R27, R29, R38, R45, R46, TAME, VOLTS1

Commit message: wenzels-real-fuzz-muff-mod release-2026-09-r6
Connections:
- net at C41.2, R42.1: now also U2.5 (+); no longer U2.3 (+)
- new net: C43.1, U2.6 (-), U2.7
Changed lines of the file:
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@@
 		(title "Wenzel’s Real Fuzz mod for classic Muff circuit")
 		(date "September 2026")
-		(rev "r5")
+		(rev "r6")
 		(comment 1 "https://www.musikding.de/Der-Muff-Triangle-Distortion-kit")
 		(comment 2 "Main Muff schematic is based on Musikding.de Muff DIY kit layout.")
@@
 		(at 379.73 87.63 0)
 		(mirror x)
-		(unit 1)
+		(unit 2)
 		(body_style 1)
 		(exclude_from_sim no)
@@
 				(path "/d1f0589a-fd5f-4fd2-a048-76dda51e2bd4"
 					(reference "U2")
-					(unit 1)
+					(unit 2)
 				)
 			)
