File: wenzels-real-fuzz-muff-mod/real-fuzz-muff-mod-for-pnp.kicad_sch (KiCad schematic)
At the start: 105 parts, among them J1 Input jack, J2 Output jack, J3 9V-18V, Q1 2N3904, Q2 2N3904, Q3 2N3904, Q4 2N3904, T1 2n2369a, T2 2n2369a, T3 2n2369a, T4 2n2369a

Commit message: wenzels-real-fuzz-muff-mod release-2026-09-r4
Parts:
- removed Q1, Q2, Q3, Q4: 2N3904, Package_TO_SOT_THT:TO-92_Inline, symbol Transistor_BJT:2N3904
- removed RLED: 10k, symbol Device:R
- removed T1, T2, T3, T4: 2n2369a, Package_TO_SOT_THT:TO-92_Inline, symbol Transistor_BJT:2N3904
- added Q1, Q2, Q3, Q4: 2N3906, Package_TO_SOT_THT:TO-92_Inline, symbol Transistor_BJT:2N3906
- added RLED1: 10k, symbol Device:R
- added T1, T2, T3, T4: Ge PNP, symbol Simulation_SPICE:PNP
Connections:
- net GND: now also C14.1, C18.1, C20.1, C23.1, C30.1, C31.1, C32.1, C33.1, C34.1, C35.1, C36.1, C37.1, C38.1, D5.1 (K), J3.2, RLED1.2; no longer C14.2, C18.2, C20.2, C23.2, C30.2, C31.2, C32.2, C33.2, C34.2, C35.2, C36.2, C37.2, C38.2, D5.2 (A), D6.1 (K), J3.1
- net at C4.1: now also Gain.2; no longer R7.1
- net at C4.2: now also R7.1; no longer Gain.2
- net at C2.1, R2.1, R3.1: now also C1.2, T1.2 (B); no longer C1.1
- net at C2.2, R3.2, R4.2: now also C3.2, T1.1 (C); no longer C3.1
- net at C10.1, C9.2, R14.2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: now also C8.2, T3.1 (C); no longer C8.1
- net at R41.1: now also C28.2, Q4.1 (E); no longer C28.1
- net at C28.2, R39.2: now also Q4.2 (B)
- net ≈-9V – ≈-18V: now reaches C21.1, R26.1, R28.2, R30.1, R32.1, R45.1
- net ≈-9V – ≈-18V: now also C14.2, C30.2, R20.1, R21.1, R32.2, R4.1, Q1.3 (C), Q2.3 (C), Q3.3 (C), Q4.3 (C); no longer C30.1
- net at C15.1, R1.2: now also C1.1; no longer C1.2
- net at C6.1, R7.2, R8.1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: now also T2.2 (B)
- net at C22.2, R21.2: now also C13.2, T4.1 (C); no longer C13.1
- net at R11.1: now also C34.2, T2.3 (E); no longer C34.1
- net at C6.2, R10.2, R9.2: now also C5.2, C7.2, T2.1 (C); no longer C5.1, C7.1
- net at R26.2, VOLTS1.1: now also C32.2, Q1.2 (B); no longer C32.1
- net at C12.2, C22.1, R19.1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: now also T4.2 (B)
- net at R5.1: now also C33.2, T1.3 (E); no longer C33.1
- net at R24.1: now also C13.1; no longer C13.2
- net at R42.1: now also C28.1; no longer C28.2
- net at R35.1, R39.1, R45.2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: now also C37.2; no longer C37.1
- net at R30.2, VOLTS2.1: now also C38.2, Q2.2 (B); no longer C38.1
- net at D6.2 (A): now also RLED1.1
- net at C12.1: now also C3.1; no longer C3.2
- net at R12.1: now also C7.1; no longer C7.2
- net at C9.1, R12.2, R13.1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: now also T3.2 (B)
- net at R29.1: now also Q1.1 (E)
- net at C25.2, R35.2: now also Q3.2 (B)
- net at R22.1: now also C36.2, T4.3 (E); no longer C36.1
- net at R16.1: now also C35.2, T3.3 (E); no longer C35.1
- net at R37.1, R38.1: now also Q3.1 (E)
- net at C19.1, R25.2, R28.1: now also C20.2; no longer C20.1
- net at R33.1: now also Q2.1 (E)
- net ≈3V–≈18V (for 18V supply) renamed ≈-3V – ≈-18V (for 18V supply)
- net ≈-3V – ≈-18V (for 18V supply): now also C23.2, C31.2; no longer C23.1, C31.1
- removed net ≈9V–≈18V: C14.1, R20.1, R21.1, R32.2, R4.1
- new net: C17.1, C18.2, D5.2 (A), D6.1 (K), J3.1, R25.1
Other:
- note added: "Negative voltage! (positive ground) PNP variant Useful for germanium PNPs Watch for electrolytic caps polarity!"
- note added: "T1, T2, T3, T4 can be for example EFT83C, they are rated -25V according to this page: https://oppermann-electronic.de/html/transistoren.html"
- moved on the sheet: C1, C13, C14, C23, C28, C3, C31, C4, C5, C7, C8, D6
