File: wenzels-colordiver-fuzz-boost/wenzels-colordiver-fuzz-boost.kicad_sch (KiCad schematic)
At the start: 85 parts, among them J1 Input jack, J2 Output jack, J3 36V, Q1 BC550, Q2 BC550, Q3 BC550, Q4 BC550, Q5 BC550, Q6 BC550, Q7 BC550

Commit message: wenzels-colordiver-fuzz-boost fixes for release-2026-08-r1
Parts:
- removed R45: 47k, symbol Device:R
- added C50: 100n, film, symbol Device:C
- added R30: 47k, symbol Device:R
- C38: value 10u -> 22u
- C39: value 500p -> 220p
- C40, C46: value 25u -> 22u
- C41, C45: value 4u7 -> 10u
- R53: value 100k -> 120k
- renumbered Bass to BASS, Gain to GAIN, Treble to TREBLE, Volume to VOLUME
Connections:
- net V+: now also R30.1
- net Vbias: now also R30.2
- net at BASS.1, R60.1: now also C50.2
- net at C44.2, R60.2: now also C45.2; no longer C45.1
- net at BASS.3, R50.2: now also C50.1
- net at C38.1, Q1.3 (E), R51.1: no longer R57.2
- net at C47.1, Q3.1 (C), R63.2: now also C45.1; no longer C45.2
- net at C38.2, GAIN.3: now also R57.2
Other:
- moved on the sheet: C35, C36, C37, C38, C39, C40, C41, C45, GAIN, J1, Q1, Q2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
