File: wenzels-colordiver-fuzz-boost/wenzels-colordiver-fuzz-boost.kicad_sch (KiCad schematic)
At the start: 86 parts, among them J1 Input jack, J2 Output jack, J3 36V, Q1 BC550, Q2 BC550, Q3 BC550, Q4 BC550, Q5 BC550, Q6 BC550, Q7 BC550

Commit message: wenzels-colordiver-fuzz-boost release-2026-09-r2
Parts:
- removed D5: 1N5819, Diode_THT:D_DO-41_SOD81_P10.16mm_Horizontal, symbol Diode:1N5819
- removed D6: LED, symbol Device:LED
- added C26, C53: 100n, film, symbol Device:C
- added C51: 100p, ceramic, symbol Device:C
- added C52: 47u, electrolytic, symbol Device:C_Polarized
- added D1: 1N4007, Diode_THT:D_DO-41_SOD81_P10.16mm_Horizontal, symbol Diode:1N4007
- added D2: LED, symbol Device:LED
- added L1: 10mH, symbol Device:L_Small
- added R31: 1, symbol Device:R
- J3: value 36V -> 18-36V
Connections:
- net GND: now also C26.2, C52.2, C53.2, D1.2 (A), D2.1 (K)
- net Vbias: now also C26.1
- net at Q7.2 (B), R26.2, VOLTS.1: now also C52.1, C53.1
- net at C17.1, C18.1, J3.2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: now also D1.1 (K), R31.1; no longer R25.1
- net at C36.2, Q1.2 (B), R56.2: now also C51.1
- net at C39.1, Q1.1 (C), Q2.2 (B)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: now also C51.2
- net at RLED.2: now also D2.2 (A)
- new net: L1.1, R31.2
- new net: L1.2, R25.1
Other:
- note added: "Optional"
- moved on the sheet: C19, C20, C21, C22, C23, C30, C37, Q7, R25, R26, R27, R28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
