File: wenzels-colormystic-fuzz-boost/wenzels-colormystic-fuzz-boost.kicad_sch (KiCad schematic)
At the start: 101 parts, among them J1 Input jack, J2 Output jack, J3 36V, Q1 BC550, Q2 BC550, Q3 BC550, Q4 BC550, Q5 BC550, Q6 BC550, Q7 BC550, Q8 BC550

Commit message: wenzels-colormystic-fuzz-boost release-2026-09-r2
Parts:
- removed C32: 10u, electrolytic, symbol Device:C_Polarized
- added C32: 3u3, film, symbol Device:C
- added L1: 10mH, symbol Device:L_Small
- added R31: 1, symbol Device:R
Connections:
- net at R43.1: now also C32.2
- net at Q7.3 (E), R70.1: now also C32.1
- net at C17.1, C18.1, D5.1 (K)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: now also R31.1; no longer R25.1
- new net: L1.1, R31.2
- new net: L1.2, R25.1
Other:
- note added: "Optional"
- moved on the sheet: C17, C18, C19, C20, C21, C22, C23, C30, C37, D5, D6, J3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

Commit message: wenzels-colormystic-fuzz-boost release-2026-09-r3
Parts:
- removed D5: 1N5819, Diode_THT:D_DO-41_SOD81_P10.16mm_Horizontal, symbol Diode:1N5819
- removed FR: SW_Nidec_CAS-120A1, Button_Switch_SMD:Nidec_Copal_CAS-120A, symbol Switch:SW_Nidec_CAS-120A1
- removed R71: 10k, symbol Device:R
- added C42: 100p, ceramic, symbol Device:C
- added C53, C54: 100n, film, symbol Device:C
- added D1: 1N4007, Diode_THT:D_DO-41_SOD81_P10.16mm_Horizontal, symbol Diode:1N4007
- C46: value 22u -> 47u
- J3: value 36V -> 18-36V
- renumbered D6 to D2
Connections:
- net GND: now also C53.2, C54.2, D1.2 (A)
- net Vbias: now also C54.1
- net at C52.1: now also Q3.3 (E), R64.1
- net at Q8.2 (B), R26.2, VOLTS.1: now also C46.1, C53.1
- net at C17.1, C18.1, J3.2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: now also D1.1 (K)
- net at C36.2, Q1.2 (B), R56.2: now also C42.1
- net at C39.1, Q1.1 (C), Q2.2 (B)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: now also C42.2
Other:
- moved on the sheet: C22, C23, C37, C52, Q8, R26, R27, R29, R30, R46, R62, R64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

Commit message: wenzels-colormystic-fuzz-boost release-2026-09-r4
Parts:
- GAIN: value C10k -> C5k
Changed lines of the file:
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@@
 		(title "Wenzel’s ColorMystic Fuzz/Boost")
 		(date "September 2026")
-		(rev "r3")
+		(rev "r4")
 		(company "Wenzel’s ColorDiver but with Quantum Mystic tone stack and extra TAME knob.")
 	)
@@
 			)
 		)
-		(property "Value" "C10k"
+		(property "Value" "C5k"
 			(at 110.49 166.3699 0)
 			(show_name no)
