File: guitar-preamps/wenzels-f-pedal-platform-preamp/wenzels-f-pedal-platform-preamp.kicad_sch (KiCad schematic)
At the start: 79 parts, among them J1 DC jack 18V, J2 DC jack 18V, J3 Input-L, J4 Input-R, J5 Output-L, J6 Output-R, U1 TL072, U2 TL072, U3 TL072

Commit message: wenzels-f-pedal-platform-preamp release-2026-09-r2
Parts:
- removed C10, C11: 100n, symbol Device:C
- removed U3: TL072, symbol Amplifier_Operational:TL072
- added R27, R28: 100, symbol Device:R
- BOOST-L, BOOST-R: value C50k -> A50k
- C30, C31: value 1n -> 47n
Connections:
- net at C20.2, VOLUME-L.2: now also R27.1; no longer U1.5 (+)
- net at C29.2, VOLUME-R.2: now also R28.1; no longer U2.5 (+)
- new net: R27.2, U1.5 (+)
- new net: R28.2, U2.5 (+)
Other:
- moved on the sheet: BOOST-L, BOOST-R, C30, C31, C32, C33, J5, J6, R23, R24, R25, R26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
