File: wenzels-dee-ass-won-guitar-distortion-pedal/wenzels-dee-ass-won-japan.kicad_sch (KiCad schematic)
At the start: 77 parts, among them J1 DC jack 18V, J2 Input, J3 Output, Q1 J113, Q2 C2240, Q3 J113, U1 TL072, U2 TA7136P

Commit message: wenzels-dee-ass-won release-2026-09-r2
Parts:
- TONE: value B25k -> B20k
Changed lines of the file:
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@@
 		(title "Wenzel’s DEE-ASS-WON (Japan variant)")
 		(date "September 2026")
-		(rev "r1")
+		(rev "r2")
 		(company "Guitar distortion pedal")
-		(comment 1 "Early Japan version that uses TA7136P preamp chip")
+		(comment 1 "Early Japan version that uses TA7136 preamp chip")
 	)
 	(junction
@@
 		(dnp no)
 		(property "Reference" "U1"
-			(at 120.65 36.322 0)
+			(at 120.65 38.608 0)
 			(show_name no)
 			(do_not_autoplace no)
@@
 		)
 		(property "Value" "TL072"
-			(at 120.65 40.894 0)
+			(at 120.65 40.132 0)
 			(show_name no)
 			(do_not_autoplace no)
@@
 		(fields_autoplaced yes)
 		(property "Reference" "TONE"
-			(at 215.9 78.7401 0)
+			(at 215.9 76.1999 0)
 			(show_name no)
 			(do_not_autoplace no)
@@
 			)
 		)
-		(property "Value" "B25k"
-			(at 215.9 76.2001 0)
+		(property "Value" "B20k"
+			(at 215.9 78.7399 0)
 			(show_name no)
 			(do_not_autoplace no)

Commit message: dee-ass-won release-2026-09-r3
Parts:
- removed R34: 47k, symbol Device:R
- added C36: 100n, symbol Device:C
- added C37: 22n, symbol Device:C
- added C38: 47n, symbol Device:C
- added HM, LM: SW_SPDT, symbol Switch:SW_SPDT
Connections:
- net +4.5V: now also C38.1
- net +9V: now also U1.5 (+), C36.1
- net GND: now also C36.2
- net at C28.2, C29.2, C30.2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: now also C37.2
- net at C30.1, R32.2: now also HM.1 (A)
- net at R30.2, TONE.1: now also LM.2 (B); no longer C31.2
- new net: C38.2, LM.1 (A)
- new net: C31.2, LM.3 (C)
- new net: C37.1, HM.2 (B)
- no-connect marks 2 -> 3
Other:
- note added: "LM and HM mids altering switches (more overlap for LP and HP filters): - Switched to pin 3 means standard DS-1 tone stack behavior - Switched to pin 1 means less mid-scoop for the lows/highs (C37 and C38)"
- moved on the sheet: BOOST, C19, C20, C21, C22, C23, C27, C28, C29, C30, C32, C33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
